Commit message: URDF file edited, still needs work on urdf and nav2

File: src/my_bot2/urdf/robot.urdf (robot description, URDF)
Before this commit: robot my_bot, 5 links, 4 joints
Links:
- removed link camera_link
- removed link dummy_link
- added link front_left_wheel, mass 1.0; collision sphere radius=0.05; visual cylinder length=0.03 radius=0.05
- added link front_right_wheel, mass 1.0; collision sphere radius=0.05; visual cylinder length=0.03 radius=0.05
- added link rear_left_wheel, mass 1.0; collision cylinder length=0.03 radius=0.05; visual cylinder length=0.03 radius=0.05
- added link rear_right_wheel, mass 1.0; collision cylinder length=0.03 radius=0.05; visual cylinder length=0.03 radius=0.05
- link base_link: mass 5.0 -> 10.0
- link laser_frame: mass None -> 0.1
Joints:
- removed joint camera_joint
- removed joint dummy_joint
- added joint front_left_wheel_joint: type continuous, parent base_link, child front_left_wheel, origin xyz=0.175 0.165 0 rpy=-1.5708 0 0, axis 0 0 1
- added joint front_right_wheel_joint: type continuous, parent base_link, child front_right_wheel, origin xyz=0.175 -0.165 0 rpy=-1.5708 0 0, axis 0 0 1
- added joint rear_left_wheel_joint: type continuous, parent base_link, child rear_left_wheel, origin xyz=-0.175 0.165 0 rpy=-1.5708 0 0, axis 0 0 1
- added joint rear_right_wheel_joint: type continuous, parent base_link, child rear_right_wheel, origin xyz=-0.175 -0.165 0 rpy=-1.5708 0 0, axis 0 0 1
- joint base_footprint_joint: child dummy_link -> base_link
- joint lidar_joint: origin xyz=0 0 0.1 rpy=0 0 0 -> xyz=0.15 0 0.1 rpy=0 0 0

Commit message: website added with text file on how to run, and some tuning to the simulation that makes it work

File: src/my_bot2/urdf/robot.urdf (robot description, URDF)
Before this commit: robot my_bot2, 7 links, 6 joints
Links:
- link front_left_wheel: mass 1.0 -> 0.5; geometry collision sphere radius=0.048; visual cylinder length=0.03 radius=0.05
- link front_right_wheel: mass 1.0 -> 0.5; geometry collision sphere radius=0.048; visual cylinder length=0.03 radius=0.05
Joints:
- joint base_footprint_joint: origin xyz=0 0 0.05 rpy=0 0 0 -> xyz=0 0 0.09 rpy=0 0 0
- joint front_left_wheel_joint: origin xyz=0.175 0.165 0 rpy=-1.5708 0 0 -> xyz=0.175 0.165 -0.04 rpy=-1.5708 0 0
- joint front_right_wheel_joint: origin xyz=0.175 -0.165 0 rpy=-1.5708 0 0 -> xyz=0.175 -0.165 -0.04 rpy=-1.5708 0 0
- joint rear_left_wheel_joint: origin xyz=-0.175 0.165 0 rpy=-1.5708 0 0 -> xyz=-0.175 0.165 -0.04 rpy=-1.5708 0 0
- joint rear_right_wheel_joint: origin xyz=-0.175 -0.165 0 rpy=-1.5708 0 0 -> xyz=-0.175 -0.165 -0.04 rpy=-1.5708 0 0
